Commit message: 更新升降柱限位

File: split_aloha_mid_360/urdf/split_aloha_mid_360.xacro (robot description, xacro)
@@ -212,6 +212,6 @@
       link="lifting_link" />
     <axis
-      xyz="0 0 1" />
-    <limit lower="-0.6" upper="0.0" effort="100" velocity="10.0"/>
+      xyz="0 0 -1" />
+    <limit lower="0.0" upper="0.8" effort="100" velocity="10.0"/>
   </joint>
   <link
