Commit message: Modify the joint limits of the Piper

File: aloha_new_description/urdf/aloha_new.urdf (robot description, URDF)
Before this commit: robot aloha_description, 50 links, 49 joints
Joints:
- joint bl_joint1: limit lower=-2.618 upper=2.618 effort=100 velocity=3 -> lower=-2.617994 upper=2.617994 effort=100 velocity=3
- joint bl_joint2: limit lower=0 upper=3.14 effort=100 velocity=3 -> lower=0 upper=3.141593 effort=100 velocity=3
- joint bl_joint3: limit lower=-2.697 upper=0 effort=100 velocity=3 -> lower=-2.967060 upper=0 effort=100 velocity=3
- joint bl_joint4: limit lower=-1.832 upper=1.832 effort=100 velocity=3 -> lower=-1.745329 upper=1.745329 effort=100 velocity=3
- joint bl_joint5: limit lower=-1.22 upper=1.22 effort=100 velocity=3 -> lower=-1.221730 upper=1.221730 effort=100 velocity=3
- joint bl_joint6: limit lower=-3.14 upper=3.14 effort=100 velocity=3 -> lower=-2.967060 upper=2.967060 effort=100 velocity=3
- joint br_joint1: limit lower=-2.618 upper=2.618 effort=100 velocity=3 -> lower=-2.617994 upper=2.617994 effort=100 velocity=3
- joint br_joint2: limit lower=0 upper=3.14 effort=100 velocity=3 -> lower=0 upper=3.141593 effort=100 velocity=3
- joint br_joint3: limit lower=-2.697 upper=0 effort=100 velocity=3 -> lower=-2.967060 upper=0 effort=100 velocity=3
- joint br_joint4: limit lower=-1.832 upper=1.832 effort=100 velocity=3 -> lower=-1.745329 upper=1.745329 effort=100 velocity=3
- joint br_joint5: limit lower=-1.22 upper=1.22 effort=100 velocity=3 -> lower=-1.221730 upper=1.221730 effort=100 velocity=3
- joint br_joint6: limit lower=-3.14 upper=3.14 effort=100 velocity=3 -> lower=-2.967060 upper=2.967060 effort=100 velocity=3
- joint fl_joint1: limit lower=-2.618 upper=2.618 effort=100 velocity=3 -> lower=-2.617994 upper=2.617994 effort=100 velocity=3
- joint fl_joint2: limit lower=0 upper=3.14 effort=100 velocity=3 -> lower=0 upper=3.141593 effort=100 velocity=3
- joint fl_joint3: limit lower=-2.697 upper=0 effort=100 velocity=3 -> lower=-2.967060 upper=0 effort=100 velocity=3
- joint fl_joint4: limit lower=-1.832 upper=1.832 effort=100 velocity=3 -> lower=-1.745329 upper=1.745329 effort=100 velocity=3
- joint fl_joint5: limit lower=-1.22 upper=1.22 effort=100 velocity=3 -> lower=-1.221730 upper=1.221730 effort=100 velocity=3
- joint fl_joint6: limit lower=-3.14 upper=3.14 effort=100 velocity=3 -> lower=-2.967060 upper=2.967060 effort=100 velocity=3
- joint fr_joint1: limit lower=-2.618 upper=2.618 effort=100 velocity=3 -> lower=-2.617994 upper=2.617994 effort=100 velocity=3
- joint fr_joint2: limit lower=0 upper=3.14 effort=100 velocity=3 -> lower=0 upper=3.141593 effort=100 velocity=3
- joint fr_joint3: limit lower=-2.697 upper=0 effort=100 velocity=3 -> lower=-2.967060 upper=0 effort=100 velocity=3
- joint fr_joint4: limit lower=-1.832 upper=1.832 effort=100 velocity=3 -> lower=-1.745329 upper=1.745329 effort=100 velocity=3
- joint fr_joint5: limit lower=-1.22 upper=1.22 effort=100 velocity=3 -> lower=-1.221730 upper=1.221730 effort=100 velocity=3
- joint fr_joint6: limit lower=-3.14 upper=3.14 effort=100 velocity=3 -> lower=-2.967060 upper=2.967060 effort=100 velocity=3

File: aloha_new_description/urdf/aloha_new_v00.urdf (robot description, URDF)
Before this commit: robot aloha_description, 50 links, 49 joints
Joints:
- joint bl_joint1: limit lower=-2.618 upper=2.618 effort=100 velocity=3 -> lower=-2.617994 upper=2.617994 effort=100 velocity=3
- joint bl_joint2: limit lower=0 upper=3.14 effort=100 velocity=3 -> lower=0 upper=3.141593 effort=100 velocity=3
- joint bl_joint3: limit lower=-2.697 upper=0 effort=100 velocity=3 -> lower=-2.967060 upper=0 effort=100 velocity=3
- joint bl_joint4: limit lower=-1.832 upper=1.832 effort=100 velocity=3 -> lower=-1.745329 upper=1.745329 effort=100 velocity=3
- joint bl_joint5: limit lower=-1.22 upper=1.22 effort=100 velocity=3 -> lower=-1.221730 upper=1.221730 effort=100 velocity=3
- joint bl_joint6: limit lower=-3.14 upper=3.14 effort=100 velocity=3 -> lower=-2.967060 upper=2.967060 effort=100 velocity=3
- joint br_joint1: limit lower=-2.618 upper=2.618 effort=100 velocity=3 -> lower=-2.617994 upper=2.617994 effort=100 velocity=3
- joint br_joint2: limit lower=0 upper=3.14 effort=100 velocity=3 -> lower=0 upper=3.141593 effort=100 velocity=3
- joint br_joint3: limit lower=-2.697 upper=0 effort=100 velocity=3 -> lower=-2.967060 upper=0 effort=100 velocity=3
- joint br_joint4: limit lower=-1.832 upper=1.832 effort=100 velocity=3 -> lower=-1.745329 upper=1.745329 effort=100 velocity=3
- joint br_joint5: limit lower=-1.22 upper=1.22 effort=100 velocity=3 -> lower=-1.221730 upper=1.221730 effort=100 velocity=3
- joint br_joint6: limit lower=-3.14 upper=3.14 effort=100 velocity=3 -> lower=-2.967060 upper=2.967060 effort=100 velocity=3
- joint fl_joint1: limit lower=-2.618 upper=2.618 effort=100 velocity=3 -> lower=-2.617994 upper=2.617994 effort=100 velocity=3
- joint fl_joint2: limit lower=0 upper=3.14 effort=100 velocity=3 -> lower=0 upper=3.141593 effort=100 velocity=3
- joint fl_joint3: limit lower=-2.697 upper=0 effort=100 velocity=3 -> lower=-2.967060 upper=0 effort=100 velocity=3
- joint fl_joint4: limit lower=-1.832 upper=1.832 effort=100 velocity=3 -> lower=-1.745329 upper=1.745329 effort=100 velocity=3
- joint fl_joint5: limit lower=-1.22 upper=1.22 effort=100 velocity=3 -> lower=-1.221730 upper=1.221730 effort=100 velocity=3
- joint fl_joint6: limit lower=-3.14 upper=3.14 effort=100 velocity=3 -> lower=-2.967060 upper=2.967060 effort=100 velocity=3
- joint fr_joint1: limit lower=-2.618 upper=2.618 effort=100 velocity=3 -> lower=-2.617994 upper=2.617994 effort=100 velocity=3
- joint fr_joint2: limit lower=0 upper=3.14 effort=100 velocity=3 -> lower=0 upper=3.141593 effort=100 velocity=3
- joint fr_joint3: limit lower=-2.697 upper=0 effort=100 velocity=3 -> lower=-2.967060 upper=0 effort=100 velocity=3
- joint fr_joint4: limit lower=-1.832 upper=1.832 effort=100 velocity=3 -> lower=-1.745329 upper=1.745329 effort=100 velocity=3
- joint fr_joint5: limit lower=-1.22 upper=1.22 effort=100 velocity=3 -> lower=-1.221730 upper=1.221730 effort=100 velocity=3
- joint fr_joint6: limit lower=-3.14 upper=3.14 effort=100 velocity=3 -> lower=-2.967060 upper=2.967060 effort=100 velocity=3

File: aloha_new_description/urdf/aloha_tracer2 copy.xacro (robot description, xacro)
@@ -861,5 +861,5 @@
         <child link="fl_link7" />
         <axis xyz="0 0 -1" />
-        <limit lower="0" upper="0.04" effort="10" velocity="1" />
+        <limit lower="0" upper="0.05" effort="10" velocity="1" />
     </joint>
     <link name="fl_link8">
@@ -898,5 +898,5 @@
         <child link="fl_link8" />
         <axis xyz="0 0 1" />
-        <limit lower="-0.04" upper="0" effort="10" velocity="1" />
+        <limit lower="-0.05" upper="0" effort="10" velocity="1" />
     </joint>
     <!--***************************** front-right ****************************** -->
@@ -1268,5 +1268,5 @@
         <child link="fr_link7" />
         <axis xyz="0 0 -1" />
-        <limit lower="0" upper="0.04" effort="10" velocity="1" />
+        <limit lower="0" upper="0.05" effort="10" velocity="1" />
     </joint>
     <link name="fr_link8">
@@ -1305,5 +1305,5 @@
         <child link="fr_link8" />
         <axis xyz="0 0 1" />
-        <limit lower="-0.04" upper="0" effort="10" velocity="1" />
+        <limit lower="-0.05" upper="0" effort="10" velocity="1" />
     </joint>
     <!--***************************** back-left ****************************** -->
@@ -1601,5 +1601,5 @@
         <child link="bl_link7" />
         <axis xyz="0 0 -1" />
-        <limit lower="0" upper="0.04" effort="10" velocity="1" />
+        <limit lower="0" upper="0.05" effort="10" velocity="1" />
     </joint>
     <link name="bl_link8">
@@ -1638,5 +1638,5 @@
         <child link="bl_link8" />
         <axis xyz="0 0 1" />
-        <limit lower="-0.04" upper="0" effort="10" velocity="1" />
+        <limit lower="-0.05" upper="0" effort="10" velocity="1" />
     </joint>
     <!--***************************** back-right ****************************** -->
@@ -1934,5 +1934,5 @@
         <child link="br_link7" />
         <axis xyz="0 0 -1" />
-        <limit lower="0" upper="0.04" effort="10" velocity="1" />
+        <limit lower="0" upper="0.05" effort="10" velocity="1" />
     </joint>
     <link name="br_link8">
@@ -1971,5 +1971,5 @@
         <child link="br_link8" />
         <axis xyz="0 0 1" />
-        <limit lower="-0.04" upper="0" effort="10" velocity="1" />
+        <limit lower="-0.05" upper="0" effort="10" velocity="1" />
     </joint>
 </robot>

File: aloha_new_description/urdf/aloha_tracer2.urdf (robot description, URDF)
Before this commit: robot aloha_description, 47 links, 47 joints
Joints:
- joint bl_joint1: limit lower=-2.618 upper=2.618 effort=100 velocity=3 -> lower=-2.617994 upper=2.617994 effort=100 velocity=3
- joint bl_joint2: limit lower=0 upper=3.14 effort=100 velocity=3 -> lower=0 upper=3.141593 effort=100 velocity=3
- joint bl_joint3: limit lower=-2.697 upper=0 effort=100 velocity=3 -> lower=-2.967060 upper=0 effort=100 velocity=3
- joint bl_joint4: limit lower=-1.832 upper=1.832 effort=100 velocity=3 -> lower=-1.745329 upper=1.745329 effort=100 velocity=3
- joint bl_joint5: limit lower=-1.22 upper=1.22 effort=100 velocity=3 -> lower=-1.221730 upper=1.221730 effort=100 velocity=3
- joint bl_joint6: limit lower=-3.14 upper=3.14 effort=100 velocity=3 -> lower=-2.967060 upper=2.967060 effort=100 velocity=3
- joint bl_joint7: limit lower=0 upper=0.04 effort=10 velocity=1 -> lower=0 upper=0.05 effort=10 velocity=1
- joint bl_joint8: limit lower=-0.04 upper=0 effort=10 velocity=1 -> lower=-0.05 upper=0 effort=10 velocity=1
- joint br_joint1: limit lower=-2.618 upper=2.618 effort=100 velocity=3 -> lower=-2.617994 upper=2.617994 effort=100 velocity=3
- joint br_joint2: limit lower=0 upper=3.14 effort=100 velocity=3 -> lower=0 upper=3.141593 effort=100 velocity=3
- joint br_joint3: limit lower=-2.697 upper=0 effort=100 velocity=3 -> lower=-2.967060 upper=0 effort=100 velocity=3
- joint br_joint4: limit lower=-1.832 upper=1.832 effort=100 velocity=3 -> lower=-1.745329 upper=1.745329 effort=100 velocity=3
- joint br_joint5: limit lower=-1.22 upper=1.22 effort=100 velocity=3 -> lower=-1.221730 upper=1.221730 effort=100 velocity=3
- joint br_joint6: limit lower=-3.14 upper=3.14 effort=100 velocity=3 -> lower=-2.967060 upper=2.967060 effort=100 velocity=3
- joint br_joint7: limit lower=0 upper=0.04 effort=10 velocity=1 -> lower=0 upper=0.05 effort=10 velocity=1
- joint br_joint8: limit lower=-0.04 upper=0 effort=10 velocity=1 -> lower=-0.05 upper=0 effort=10 velocity=1
- joint fl_joint1: limit lower=-2.618 upper=2.618 effort=100 velocity=3 -> lower=-2.617994 upper=2.617994 effort=100 velocity=3
- joint fl_joint2: limit lower=0 upper=3.14 effort=100 velocity=3 -> lower=0 upper=3.141593 effort=100 velocity=3
- joint fl_joint3: limit lower=-2.697 upper=0 effort=100 velocity=3 -> lower=-2.967060 upper=0 effort=100 velocity=3
- joint fl_joint4: limit lower=-1.832 upper=1.832 effort=100 velocity=3 -> lower=-1.745329 upper=1.745329 effort=100 velocity=3
- joint fl_joint5: limit lower=-1.22 upper=1.22 effort=100 velocity=3 -> lower=-1.221730 upper=1.221730 effort=100 velocity=3
- joint fl_joint6: limit lower=-3.14 upper=3.14 effort=100 velocity=3 -> lower=-2.967060 upper=2.967060 effort=100 velocity=3
- joint fl_joint7: limit lower=0 upper=0.04 effort=10 velocity=1 -> lower=0 upper=0.05 effort=10 velocity=1
- joint fl_joint8: limit lower=-0.04 upper=0 effort=10 velocity=1 -> lower=-0.05 upper=0 effort=10 velocity=1
- joint fr_joint1: limit lower=-2.618 upper=2.618 effort=100 velocity=3 -> lower=-2.617994 upper=2.617994 effort=100 velocity=3
- joint fr_joint2: limit lower=0 upper=3.14 effort=100 velocity=3 -> lower=0 upper=3.141593 effort=100 velocity=3
- joint fr_joint3: limit lower=-2.697 upper=0 effort=100 velocity=3 -> lower=-2.967060 upper=0 effort=100 velocity=3
- joint fr_joint4: limit lower=-1.832 upper=1.832 effort=100 velocity=3 -> lower=-1.745329 upper=1.745329 effort=100 velocity=3
- joint fr_joint5: limit lower=-1.22 upper=1.22 effort=100 velocity=3 -> lower=-1.221730 upper=1.221730 effort=100 velocity=3
- joint fr_joint6: limit lower=-3.14 upper=3.14 effort=100 velocity=3 -> lower=-2.967060 upper=2.967060 effort=100 velocity=3
- joint fr_joint7: limit lower=0 upper=0.04 effort=10 velocity=1 -> lower=0 upper=0.05 effort=10 velocity=1
- joint fr_joint8: limit lower=-0.04 upper=0 effort=10 velocity=1 -> lower=-0.05 upper=0 effort=10 velocity=1

File: aloha_new_description/urdf/aloha_tracer2_d435.urdf (robot description, URDF)
Before this commit: robot aloha_description, 58 links, 57 joints
Joints:
- joint bl_joint1: limit lower=-2.618 upper=2.618 effort=100 velocity=3 -> lower=-2.617994 upper=2.617994 effort=100 velocity=3
- joint bl_joint2: limit lower=0 upper=3.14 effort=100 velocity=3 -> lower=0 upper=3.141593 effort=100 velocity=3
- joint bl_joint3: limit lower=-2.697 upper=0 effort=100 velocity=3 -> lower=-2.967060 upper=0 effort=100 velocity=3
- joint bl_joint4: limit lower=-1.832 upper=1.832 effort=100 velocity=3 -> lower=-1.745329 upper=1.745329 effort=100 velocity=3
- joint bl_joint5: limit lower=-1.22 upper=1.22 effort=100 velocity=3 -> lower=-1.221730 upper=1.221730 effort=100 velocity=3
- joint bl_joint6: limit lower=-3.14 upper=3.14 effort=100 velocity=3 -> lower=-2.967060 upper=2.967060 effort=100 velocity=3
- joint bl_joint7: limit lower=0 upper=0.04 effort=10 velocity=1 -> lower=0 upper=0.05 effort=10 velocity=1
- joint bl_joint8: limit lower=-0.04 upper=0 effort=10 velocity=1 -> lower=-0.05 upper=0 effort=10 velocity=1
- joint br_joint1: limit lower=-2.618 upper=2.618 effort=100 velocity=3 -> lower=-2.617994 upper=2.617994 effort=100 velocity=3
- joint br_joint2: limit lower=0 upper=3.14 effort=100 velocity=3 -> lower=0 upper=3.141593 effort=100 velocity=3
- joint br_joint3: limit lower=-2.697 upper=0 effort=100 velocity=3 -> lower=-2.967060 upper=0 effort=100 velocity=3
- joint br_joint4: limit lower=-1.832 upper=1.832 effort=100 velocity=3 -> lower=-1.745329 upper=1.745329 effort=100 velocity=3
- joint br_joint5: limit lower=-1.22 upper=1.22 effort=100 velocity=3 -> lower=-1.221730 upper=1.221730 effort=100 velocity=3
- joint br_joint6: limit lower=-3.14 upper=3.14 effort=100 velocity=3 -> lower=-2.967060 upper=2.967060 effort=100 velocity=3
- joint br_joint7: limit lower=0 upper=0.04 effort=10 velocity=1 -> lower=0 upper=0.05 effort=10 velocity=1
- joint br_joint8: limit lower=-0.04 upper=0 effort=10 velocity=1 -> lower=-0.05 upper=0 effort=10 velocity=1
- joint fl_joint1: limit lower=-2.618 upper=2.618 effort=100 velocity=3 -> lower=-2.617994 upper=2.617994 effort=100 velocity=3
- joint fl_joint2: limit lower=0 upper=3.14 effort=100 velocity=3 -> lower=0 upper=3.141593 effort=100 velocity=3
- joint fl_joint3: limit lower=-2.697 upper=0 effort=100 velocity=3 -> lower=-2.967060 upper=0 effort=100 velocity=3
- joint fl_joint4: limit lower=-1.832 upper=1.832 effort=100 velocity=3 -> lower=-1.745329 upper=1.745329 effort=100 velocity=3
- joint fl_joint5: limit lower=-1.22 upper=1.22 effort=100 velocity=3 -> lower=-1.221730 upper=1.221730 effort=100 velocity=3
- joint fl_joint6: limit lower=-3.14 upper=3.14 effort=100 velocity=3 -> lower=-2.967060 upper=2.967060 effort=100 velocity=3
- joint fl_joint7: limit lower=0 upper=0.04 effort=10 velocity=1 -> lower=0 upper=0.05 effort=10 velocity=1
- joint fl_joint8: limit lower=-0.04 upper=0 effort=10 velocity=1 -> lower=-0.05 upper=0 effort=10 velocity=1
- joint fr_joint1: limit lower=-2.618 upper=2.618 effort=100 velocity=3 -> lower=-2.617994 upper=2.617994 effort=100 velocity=3
- joint fr_joint2: limit lower=0 upper=3.14 effort=100 velocity=3 -> lower=0 upper=3.141593 effort=100 velocity=3
- joint fr_joint3: limit lower=-2.697 upper=0 effort=100 velocity=3 -> lower=-2.967060 upper=0 effort=100 velocity=3
- joint fr_joint4: limit lower=-1.832 upper=1.832 effort=100 velocity=3 -> lower=-1.745329 upper=1.745329 effort=100 velocity=3
- joint fr_joint5: limit lower=-1.22 upper=1.22 effort=100 velocity=3 -> lower=-1.221730 upper=1.221730 effort=100 velocity=3
- joint fr_joint6: limit lower=-3.14 upper=3.14 effort=100 velocity=3 -> lower=-2.967060 upper=2.967060 effort=100 velocity=3
- joint fr_joint7: limit lower=0 upper=0.04 effort=10 velocity=1 -> lower=0 upper=0.05 effort=10 velocity=1
- joint fr_joint8: limit lower=-0.04 upper=0 effort=10 velocity=1 -> lower=-0.05 upper=0 effort=10 velocity=1

File: aloha_new_description/urdf/aloha_tracer2_d435_dark.urdf (robot description, URDF)
Before this commit: robot aloha_description, 58 links, 57 joints
Joints:
- joint bl_joint1: limit lower=-2.618 upper=2.618 effort=100 velocity=3 -> lower=-2.617994 upper=2.617994 effort=100 velocity=3
- joint bl_joint2: limit lower=0 upper=3.14 effort=100 velocity=3 -> lower=0 upper=3.141593 effort=100 velocity=3
- joint bl_joint3: limit lower=-2.697 upper=0 effort=100 velocity=3 -> lower=-2.967060 upper=0 effort=100 velocity=3
- joint bl_joint4: limit lower=-1.832 upper=1.832 effort=100 velocity=3 -> lower=-1.745329 upper=1.745329 effort=100 velocity=3
- joint bl_joint5: limit lower=-1.22 upper=1.22 effort=100 velocity=3 -> lower=-1.221730 upper=1.221730 effort=100 velocity=3
- joint bl_joint6: limit lower=-3.14 upper=3.14 effort=100 velocity=3 -> lower=-2.967060 upper=2.967060 effort=100 velocity=3
- joint bl_joint7: limit lower=0 upper=0.04 effort=10 velocity=1 -> lower=0 upper=0.05 effort=10 velocity=1
- joint bl_joint8: limit lower=-0.04 upper=0 effort=10 velocity=1 -> lower=-0.05 upper=0 effort=10 velocity=1
- joint br_joint1: limit lower=-2.618 upper=2.618 effort=100 velocity=3 -> lower=-2.617994 upper=2.617994 effort=100 velocity=3
- joint br_joint2: limit lower=0 upper=3.14 effort=100 velocity=3 -> lower=0 upper=3.141593 effort=100 velocity=3
- joint br_joint3: limit lower=-2.697 upper=0 effort=100 velocity=3 -> lower=-2.967060 upper=0 effort=100 velocity=3
- joint br_joint4: limit lower=-1.832 upper=1.832 effort=100 velocity=3 -> lower=-1.745329 upper=1.745329 effort=100 velocity=3
- joint br_joint5: limit lower=-1.22 upper=1.22 effort=100 velocity=3 -> lower=-1.221730 upper=1.221730 effort=100 velocity=3
- joint br_joint6: limit lower=-3.14 upper=3.14 effort=100 velocity=3 -> lower=-2.967060 upper=2.967060 effort=100 velocity=3
- joint br_joint7: limit lower=0 upper=0.04 effort=10 velocity=1 -> lower=0 upper=0.05 effort=10 velocity=1
- joint br_joint8: limit lower=-0.04 upper=0 effort=10 velocity=1 -> lower=-0.05 upper=0 effort=10 velocity=1
- joint fl_joint1: limit lower=-2.618 upper=2.618 effort=100 velocity=3 -> lower=-2.617994 upper=2.617994 effort=100 velocity=3
- joint fl_joint2: limit lower=0 upper=3.14 effort=100 velocity=3 -> lower=0 upper=3.141593 effort=100 velocity=3
- joint fl_joint3: limit lower=-2.697 upper=0 effort=100 velocity=3 -> lower=-2.967060 upper=0 effort=100 velocity=3
- joint fl_joint4: limit lower=-1.832 upper=1.832 effort=100 velocity=3 -> lower=-1.745329 upper=1.745329 effort=100 velocity=3
- joint fl_joint5: limit lower=-1.22 upper=1.22 effort=100 velocity=3 -> lower=-1.221730 upper=1.221730 effort=100 velocity=3
- joint fl_joint6: limit lower=-3.14 upper=3.14 effort=100 velocity=3 -> lower=-2.967060 upper=2.967060 effort=100 velocity=3
- joint fl_joint7: limit lower=0 upper=0.04 effort=10 velocity=1 -> lower=0 upper=0.05 effort=10 velocity=1
- joint fl_joint8: limit lower=-0.04 upper=0 effort=10 velocity=1 -> lower=-0.05 upper=0 effort=10 velocity=1
- joint fr_joint1: limit lower=-2.618 upper=2.618 effort=100 velocity=3 -> lower=-2.617994 upper=2.617994 effort=100 velocity=3
- joint fr_joint2: limit lower=0 upper=3.14 effort=100 velocity=3 -> lower=0 upper=3.141593 effort=100 velocity=3
- joint fr_joint3: limit lower=-2.697 upper=0 effort=100 velocity=3 -> lower=-2.967060 upper=0 effort=100 velocity=3
- joint fr_joint4: limit lower=-1.832 upper=1.832 effort=100 velocity=3 -> lower=-1.745329 upper=1.745329 effort=100 velocity=3
- joint fr_joint5: limit lower=-1.22 upper=1.22 effort=100 velocity=3 -> lower=-1.221730 upper=1.221730 effort=100 velocity=3
- joint fr_joint6: limit lower=-3.14 upper=3.14 effort=100 velocity=3 -> lower=-2.967060 upper=2.967060 effort=100 velocity=3
- joint fr_joint7: limit lower=0 upper=0.04 effort=10 velocity=1 -> lower=0 upper=0.05 effort=10 velocity=1
- joint fr_joint8: limit lower=-0.04 upper=0 effort=10 velocity=1 -> lower=-0.05 upper=0 effort=10 velocity=1
